File: KiCad/Hex Display Expansion/_autosave-AT_HEX.kicad_pcb (KiCad board)
At the start: 2 copper layers, 101.1 x 77.4 mm, 38 parts, among them J1 Expansion Connector, J2 PWR, Q1 BC557, Q2 BC557, Q3 BC557, Q4 BC557, Q5 BC557, Q6 BC557, U1 NE555P, U10 HDSP-7801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

Commit message: Silk Screen Modifications - Hex Display WIP
Parts:
- removed the REF** at (111.7, 63.6)
- moved REF** 2.24 mm to (127.0, 88.3)
Routing:
- net /~Q0: track 26.6 -> 49.4 mm, vias 0 -> 1
- net /Q1: track 18.4 -> 31.6 mm, vias 0 -> 1
- net EN_H: track 110.7 -> 112.7 mm
- net HEX2: track 106.4 -> 107.8 mm
- net (no net): vias 1 -> 0
Other:
- board text removed: "+3.3V"
- board text removed: "+5V"
- board text removed: "A00"
- board text removed: "A01"
- board text removed: "A02"
- board text removed: "A03"
- board text removed: "A04"
- board text removed: "A05"
- board text removed: "A06"
- board text removed: "A07"
- board text removed: "A08"
- board text removed: "A09"
- board text removed: "A10"
- board text removed: "A11"
- board text removed: "A12"
- board text removed: "A13"
- board text removed: "A14"
- board text removed: "A15"
- board text removed: "Based on Ben Eater’s 6502 project and"
- board text removed: "CLK"
- board text removed: "D0"
- board text removed: "D1"
- board text removed: "D2"
- board text removed: "D3"
- board text removed: "D4"
- board text removed: "D5"
- board text removed: "D6"
- board text removed: "D7"
- board text removed: "GND"
- board text removed: "NC"
- board text removed: "R~W"
- board text removed: "SIGNAL"
- board text removed: "https://github.com/dbuchwald/6502"
- board text removed: "the PCB designs by Dawid Buchwald"
- board text removed: "~IOCS"
- board text removed: "~IRQ"
- board text removed: "~RES"
- board text removed: "~ROMCS"
- board text removed: "~ROMOE"
