File: KiCad/Hex Display Expansion/16 bit Hex.sch (KiCad schematic (older format))
At the start: 15 parts, among them Q3 BC557, Q4 BC557, Q5 BC557, Q6 BC557, U10 HDSP-7801, U11 HDSP-7801, U12 HDSP-7801, U7 74HC04, U8 GAL16V8, U9 HDSP-7801

Commit message: HEX Board Mods
Hex board changes. Main board Hex to Latches
Parts:
- added unit 5 of U7
- added unit 6 of U7
- U10, U11, U12, U9: symbol Display_Character:HDSP-7801 -> Display_Character:HDSP-7801_test
Connections:
- wire segments 135 -> 138
- no-connect marks 10 -> 12
Changed lines of the file:
@@
 	7150 3425 7250 3425
 $Comp
-L Display_Character:HDSP-7801 U?
+L Display_Character:HDSP-7801_test U?
 U 1 1 63CE3723
 P 6850 3125
@@
 $EndComp
 $Comp
-L Display_Character:HDSP-7801 U?
+L Display_Character:HDSP-7801_test U?
 U 1 1 63CE3729
 P 5475 3125
@@
 	8575 3425 8650 3425
 $Comp
-L Display_Character:HDSP-7801 U?
+L Display_Character:HDSP-7801_test U?
 U 1 1 63CE374E
 P 8275 3125
@@
 $EndComp
 $Comp
-L Display_Character:HDSP-7801 U?
+L Display_Character:HDSP-7801_test U?
 U 1 1 63CE3754
 P 9650 3125
@@
 Connection ~ 8650 3425
 Connection ~ 10025 3425
+NoConn ~ 2150 1050
+$Comp
+L 74xx:74HC04 U7
+U 6 1 637C9A2B
+P 1850 1600
+F 0 "U7" H 1850 1917 50  0000 C CNN
+F 1 "74HC04" H 1850 1826 50  0000 C CNN
+F 2 "Package_DIP:DIP-14_W7.62mm_Socket" H 1850 1600 50  0001 C CNN
+F 3 "https://assets.nexperia.com/documents/data-sheet/74HC_HCT04.pdf" H 1850 1600 50  0001 C CNN
+	6    1850 1600
+	1    0    0    -1
+$EndComp
+NoConn ~ 2150 1600
+Wire Wire Line
+	1550 1050 1550 1325
+Wire Wire Line
+	1225 1325 1550 1325
 Wire Bus Line
 	1725 2775 1725 3425
+Connection ~ 1550 1325
+Wire Wire Line
+	1550 1325 1550 1600
+$Comp
+L power:GND #PWR?
+U 1 1 637DBD84
+P 1225 1325
+F 0 "#PWR?" H 1225 1075 50  0001 C CNN
+F 1 "GND" H 1230 1152 50  0000 C CNN
+F 2 "" H 1225 1325 50  0001 C CNN
+F 3 "" H 1225 1325 50  0001 C CNN
+	1    1225 1325
+	1    0    0    -1
+$EndComp
+$Comp
+L 74xx:74HC04 U7
+U 5 1 637B7F5F
+P 1850 1050
+F 0 "U7" H 1850 1367 50  0000 C CNN
+F 1 "74HC04" H 1850 1276 50  0000 C CNN
+F 2 "Package_DIP:DIP-14_W7.62mm_Socket" H 1850 1050 50  0001 C CNN
+F 3 "https://assets.nexperia.com/documents/data-sheet/74HC_HCT04.pdf" H 1850 1050 50  0001 C CNN
+	5    1850 1050
+	1    0    0    -1
+$EndComp
 $EndSCHEMATC
