File: KiCad/Hex Display Expansion/AT_HEX.sch (KiCad schematic (older format))
At the start: 11 parts, among them J1 Expansion Connector, J2 PWR, U1 NE555P, U13 74HC244, U14 74HC244, U5 74HC74, U6 74HC00

Commit message: HEX Board Mods
Hex board changes. Main board Hex to Latches
Parts:
- removed D1: D, Diode_THT:D_DO-15_P10.16mm_Horizontal, symbol Device:D
- removed J2: PWR, Connector_PinHeader_2.54mm:PinHeader_1x02_P2.54mm_Vertical, symbol Connector_Generic:Conn_01x02
- removed U13, U14: 74HC244, Package_DIP:DIP-20_W7.62mm_Socket, symbol 74xx:74HC244
- removed U5: 74HC74, Package_DIP:DIP-14_W7.62mm_Socket, symbol 74xx:74HC74
- removed U6: 74HC00, Package_DIP:DIP-14_W7.62mm_Socket, symbol 74xx:74HC00
- added C2, C3, C4: 100n, Capacitor_THT:C_Disc_D5.0mm_W2.5mm_P5.00mm, symbol Device:C
- added C5: 0.01uF, Capacitor_THT:C_Disc_D5.0mm_W2.5mm_P5.00mm, symbol Device:C
- added J2: Conn_02x03_Odd_Even, Connector_PinSocket_2.54mm:PinSocket_2x03_P2.54mm_Vertical, symbol Connector_Generic:Conn_02x03_Odd_Even
- added J3: Conn_01x03, Connector_PinHeader_2.54mm:PinHeader_1x03_P2.54mm_Vertical, symbol Connector_Generic:Conn_01x03
- added Q1, Q2, Q3, Q4, Q5, Q6: BC557, Package_TO_SOT_THT:TO-92_Inline, symbol Transistor_BJT:BC557
- added R10, R11, R12, R13, R14, R17, R7, R8, R9: 4k7, Resistor_THT:R_Axial_DIN0207_L6.3mm_D2.5mm_P7.62mm_Horizontal, symbol Device:R
- added R15, R16, R18: 2k2, Resistor_THT:R_Axial_DIN0207_L6.3mm_D2.5mm_P7.62mm_Horizontal, symbol Device:R
- added RN1, RN2, RN3: 100, Package_DIP:DIP-16_W7.62mm_Socket, symbol Device:R_Pack08
- added RV1, RV2: R_POT_Small, Potentiometer_THT:Potentiometer_Piher_PT-10-V10_Vertical, symbol Device:R_POT_Small
- added U10, U5, U6, U7, U8, U9: E10561, Display_7Segment:7SegmentLED_LTS6760_LTS6780, symbol Display_Character:LuckyLight_KWI-561AVB
- added U2, U3, U4: GAL16V8, Package_DIP:DIP-20_W7.62mm_Socket, symbol Logic_Programmable:GAL16V8
- C1: value 68n -> 0.01uF
- J1: footprint Connector_PinHeader_2.54mm:PinHeader_2x12_P2.54mm_Vertical -> Connector_PinHeader_2.54mm:PinHeader_2x16_P2.54mm_Vertical; symbol Connector_Generic:Conn_02x12_Odd_Even -> Connector_Generic:Conn_02x16_Odd_Even
- R1: value 51k -> 1k
- R2: value 51k -> 100k
Connections:
- net +5V: now also C2.1, C3.1, C4.1, J3.2 (Pin_2), RV1.1, RV2.1, U2.20 (VCC), U3.20 (VCC), U4.20 (VCC); no longer R2.1, U1.4 (R)
- net EN_H: now also R13.2, R17.2, R9.2, U2.1 (I1/CLK), U3.1 (I1/CLK), U4.1 (I1/CLK)
- net GND: now also J1.30 (Pin_30), J1.32 (Pin_32), C2.2, C3.2, C4.2, C5.2, J2.5 (Pin_5), R11.1, R12.1, R15.2, R16.2, R7.1, R8.1, U3.10 (GND), U4.10 (GND)
- net a0: now also U3.2 (I2)
- net a1: now also U3.3 (I3)
- net a10: now also U4.4 (I4)
- net a11: now also U4.5 (I5)
- net a12: now also U4.6 (I6)
- net a13: now also U4.7 (I7)
- net a14: now also U4.8 (I8)
- net a15: now also U4.9 (I9)
- net a2: now also U3.4 (I4)
- net a3: now also U3.5 (I5)
- net a4: now also U3.6 (I6)
- net a5: now also U3.7 (I7)
- net a6: now also U3.8 (I8)
- net a7: now also U3.9 (I9)
- net a8: now also U4.2 (I2)
- net a9: now also U4.3 (I3)
- net d0: now also U2.9 (I9)
- net d1: now also U2.8 (I8)
- net d2: now also U2.7 (I7)
- net d3: now also U2.6 (I6)
- net d4: now also U2.5 (I5)
- net d5: now also U2.4 (I4)
- net d6: now also U2.3 (I3)
- net d7: now also U2.2 (I2)
- net at U1.5 (CV): now also C5.1
- net at R1.2, U1.7 (DIS): now also R2.1
- new net: J1.31 (Pin_31), J3.1 (Pin_1)
- new net: R15.1, U9.8 (CA)
- new net: R16.1, U10.8 (CA)
- new net: Q5.1 (C), Q6.1 (C), RV2.2
- new net: Q5.2 (B), R17.1
- new net: Q5.3 (E), U9.3 (CA)
- new net: Q6.2 (B), R18.1
- new net: Q6.3 (E), U10.3 (CA)
- new net: RN1.1 (R1.1), U2.18 (IO2)
- new net: RN1.10 (R7.2), U10.10 (G), U9.10 (G)
- new net: RN1.11 (R6.2), U10.9 (F), U9.9 (F)
- new net: RN1.12 (R5.2), U10.1 (E), U9.1 (E)
- new net: RN1.13 (R4.2), U10.2 (D), U9.2 (D)
- new net: RN1.14 (R3.2), U10.4 (C), U9.4 (C)
- new net: RN1.15 (R2.2), U10.6 (B), U9.6 (B)
- new net: RN1.16 (R1.2), U10.7 (A), U9.7 (A)
- new net: RN1.2 (R2.1), U2.17 (I03)
- new net: RN1.3 (R3.1), U2.16 (IO4)
- new net: RN1.4 (R4.1), U2.15 (IO5)
- new net: RN1.5 (R5.1), U2.14 (IO6)
- new net: RN1.6 (R6.1), U2.13 (IO7)
- new net: RN1.7 (R7.1), U2.12 (IO8)
- new net: RN2.7 (R7.1), U3.12 (IO8)
- new net: RN2.6 (R6.1), U3.13 (IO7)
- new net: RN2.5 (R5.1), U3.14 (IO6)
- new net: RN2.4 (R4.1), U3.15 (IO5)
- new net: RN2.3 (R3.1), U3.16 (IO4)
- new net: RN2.2 (R2.1), U3.17 (I03)
- new net: RN2.1 (R1.1), U3.18 (IO2)
- new net: R7.2, U7.8 (CA)
- new net: R8.2, U8.8 (CA)
- new net: Q1.1 (C), Q2.1 (C), Q3.1 (C), Q4.1 (C), RV1.2
- new net: Q1.2 (B), R9.1
- new net: Q1.3 (E), U7.3 (CA)
- new net: Q2.2 (B), R10.1
- new net: Q2.3 (E), U8.3 (CA)
- new net: RN2.10 (R7.2), U7.10 (G), U8.10 (G)
- new net: RN2.11 (R6.2), U7.9 (F), U8.9 (F)
- new net: RN2.12 (R5.2), U7.1 (E), U8.1 (E)
- new net: RN2.13 (R4.2), U7.2 (D), U8.2 (D)
- new net: RN2.14 (R3.2), U7.4 (C), U8.4 (C)
- new net: RN2.15 (R2.2), U7.6 (B), U8.6 (B)
- new net: RN2.16 (R1.2), U7.7 (A), U8.7 (A)
- new net: Q4.2 (B), R14.1
- new net: Q4.3 (E), U6.3 (CA)
- new net: Q3.2 (B), R13.1
- new net: Q3.3 (E), U5.3 (CA)
- new net: RN3.7 (R7.1), U4.12 (IO8)
- new net: RN3.6 (R6.1), U4.13 (IO7)
- new net: RN3.5 (R5.1), U4.14 (IO6)
- new net: RN3.4 (R4.1), U4.15 (IO5)
- new net: RN3.3 (R3.1), U4.16 (IO4)
- new net: RN3.2 (R2.1), U4.17 (I03)
- new net: RN3.1 (R1.1), U4.18 (IO2)
- new net: R11.2, U5.8 (CA)
- new net: R12.2, U6.8 (CA)
- new net: RN3.10 (R7.2), U5.10 (G), U6.10 (G)
- new net: RN3.11 (R6.2), U5.9 (F), U6.9 (F)
- new net: RN3.12 (R5.2), U5.1 (E), U6.1 (E)
- new net: RN3.13 (R4.2), U5.2 (D), U6.2 (D)
- new net: RN3.14 (R3.2), U5.4 (C), U6.4 (C)
- new net: RN3.15 (R2.2), U5.6 (B), U6.6 (B)
- new net: RN3.16 (R1.2), U5.7 (A), U6.7 (A)
- new net +3.3V: J1.29 (Pin_29), J2.6 (Pin_6)
- new net EN_DL: R18.2, U2.19 (IO1)
- new net EN_a0L: R10.2, U3.19 (IO1)
- new net EN_a8L: R14.2, U4.19 (IO1)
- new net ~RAM_CS: J1.28 (Pin_28), J2.3 (Pin_3)
- new net ~ROM_CS: J1.26 (Pin_26), J2.1 (Pin_1)
- new net ~ROM_OE: J1.25 (Pin_25), J2.2 (Pin_2)
- no-connect marks 1 -> 21
Other:
- moved on the sheet: C1, R1, R2, U1
