File: KiCad/Rev002/AT_65C02_Computer/AT_65C02_Computer_Rev002.sch (KiCad schematic (older format))
At the start: 33 parts, among them J1 CLK Jumper, J7 Expansion port, SW4 SW_SPDT, U1 74HC21, U2 74HC00, U3 74HC02, U4 NE555, U7 65C02S, U8 28C256, U9 62256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

Commit message: HEX Board Mods
Hex board changes. Main board Hex to Latches
Parts:
- added JP11: ~OE Low Fixed, Connector_PinHeader_2.54mm:PinHeader_1x02_P2.54mm_Vertical, symbol Jumper:Jumper_2_Open
Connections:
- net labels added: ~RAM_OE
- wire segments 306 -> 307
Changed lines of the file:
@@
 $Descr A4 11693 8268
 encoding utf-8
-Sheet 1 8
+Sheet 1 7
 Title "AT_65C02 Hobby Computer"
 Date ""
@@
 Wire Wire Line
 	4450 4350 4350 4350
-Wire Wire Line
-	4750 4250 4750 4950
-Wire Wire Line
-	4750 4950 4350 4950
 Text Label 4500 5250 2    50   ~ 0
 d7
@@
 a13
 Wire Wire Line
-	4750 4950 4750 5150
-Wire Wire Line
 	4750 5150 4350 5150
-Connection ~ 4750 4950
 Text GLabel 4600 4250 1    50   Input ~ 0
 R~W
@@
 Text GLabel 1350 2550 3    50   Input ~ 0
 GND
+Wire Wire Line
+	4750 4250 4750 5150
+Wire Wire Line
+	4350 4950 4675 4950
+Wire Wire Line
+	4675 4950 4675 5525
+Wire Wire Line
+	4675 5525 4825 5525
+Text GLabel 4825 5525 2    50   Input ~ 0
+~RAM_OE
+$Comp
+L Jumper:Jumper_2_Open JP11
+U 1 1 639E7BFF
+P 7650 4100
+F 0 "JP11" H 7650 4347 50  0000 C CNN
+F 1 "~OE Low Fixed" H 7650 4249 50  0000 C CNN
+F 2 "Connector_PinHeader_2.54mm:PinHeader_1x02_P2.54mm_Vertical" H 7650 4100 50  0001 C CNN
+F 3 "~" H 7650 4100 50  0001 C CNN
+	1    7650 4100
+	1    0    0    -1
+$EndComp
+Text GLabel 7450 4100 0    50   Input ~ 0
+~RAM_CS
+Text GLabel 7850 4100 2    50   Input ~ 0
+~RAM_OE
 Wire Bus Line
 	3100 5450 3100 5650
@@
 Wire Bus Line
 	5350 4250 5350 5750
-$Sheet
-S 10175 6300 500  150
-U 63758CB0
-F0 "Floppy" 50
-F1 "Floppy.sch" 50
-$EndSheet
 $EndSCHEMATC
