File: KiCad/Rev002/AT_65C02_Computer/Memory Decoder.sch (KiCad schematic (older format))
At the start: 3 parts, among them U29 Flexible Memory Decoder

Commit message: HEX Board Mods
Hex board changes. Main board Hex to Latches
Parts:
- added J23: Address, Connector_PinSocket_2.54mm:PinSocket_1x16_P2.54mm_Vertical, symbol Connector_Generic:Conn_01x16
- added J24: Conn_02x02_Odd_Even, Connector_PinSocket_2.54mm:PinSocket_1x04_P2.54mm_Vertical, symbol Connector_Generic:Conn_01x04
- added J25, J26: Conn_01x03, Connector_PinSocket_2.54mm:PinSocket_1x03_P2.54mm_Vertical, symbol Connector_Generic:Conn_01x03
- added JP15: V1_CS1_Select, Connector_PinHeader_2.54mm:PinHeader_1x03_P2.54mm_Vertical, symbol blinken:Jumper_Jumper_3_Bridged12
- added JP16: V2_CS1_Select, Connector_PinHeader_2.54mm:PinHeader_1x03_P2.54mm_Vertical, symbol blinken:Jumper_Jumper_3_Bridged12
- added JP17: A_CS0_Select, Connector_PinHeader_2.54mm:PinHeader_1x03_P2.54mm_Vertical, symbol blinken:Jumper_Jumper_3_Bridged12
- added JP18: V1_CS2_Select, Connector_PinHeader_2.54mm:PinHeader_1x03_P2.54mm_Vertical, symbol blinken:Jumper_Jumper_3_Bridged12
- added JP19: V2_CS2_Select, Connector_PinHeader_2.54mm:PinHeader_1x03_P2.54mm_Vertical, symbol blinken:Jumper_Jumper_3_Bridged12
- added JP20: A_CS1_Select, Connector_PinHeader_2.54mm:PinHeader_1x03_P2.54mm_Vertical, symbol blinken:Jumper_Jumper_3_Bridged12
Connections:
- net labels added: A_CSO, V1CS1, V2CS1, ~IO1, ~IOCS_A, ~IOCS_V1, ~IOCS_V2, ~RAM_CS, ~RAM_OE, ~ROM_CS, ~ROM_OE
- net labels removed: ~OE, ~RAM, ~ROM
- wire segments 21 -> 57
Other:
- moved on the sheet: JP10, R39, U29
