File: KiCad/Rev002/AT_65C02_Computer/AT_65C02_Computer_Rev002.kicad_pcb (KiCad board)
At the start: 2 copper layers, 241.3 x 149.9 mm, 155 parts, among them J1 CLK Jumper, J11 LCD Connector, J12 Expansion port #2, J14 ESP Interface, J15 Level_Shifter_HV, J16 Level_Shifter_LV, J18 CPU Signals, J19 Address Decoder Enable, J2 Optional UART Port, J20 Modem Interface, J3 Conn_01x06_Female, J4 AudioJack4, J5 Barrel_Jack-Connector, J6 Mini-DIN-6, J7 Expansion port, J8 AVR-ISP-10, J9 VIA2PA - VIA2PB, Q1 BC547, SW1 SW_SPDT, SW2 Step, SW3 Mode, SW4 SW_SPDT, U1 74HC21, U10 ATtiny4313-PU, U11 65C22S, U12 65C22S, U13 L7806, U14 74LS04, U15 74LS08, U16 74LS32, U17 NE555, U18 NE555, U19 NE555, U2 74HC00, U20 74HCT540, U21 74HCT573, U22 74HCT573, U23 74HCT573, U24 10_LED_Array, U25 10_LED_Array, U26 10_LED_Array, U27 10_LED_Array, U28 LM393, U29 Flexible Memory Decoder, U3 74HC02, U4 NE555, U5 65C51N, U6 Regulator_Linear_L7805, U7 65C02S, U8 28C256, U9 62256, X1 1MHz, X2 1.8432MHz

Commit message: HEX Board Mods
Hex board changes. Main board Hex to Latches
Parts:
- added J21: Expansion port, Connector_PinSocket_2.54mm:PinSocket_2x16_P2.54mm_Vertical, F.Cu at (11.2, 75.5)
- added J22: Expansion port, Connector_PinSocket_2.54mm:PinSocket_2x16_P2.54mm_Vertical, F.Cu at (31.4, 75.5)
- added J23: Address, Connector_PinSocket_2.54mm:PinSocket_1x16_P2.54mm_Vertical, F.Cu at (35.7, 131.5)
- added J24: Conn_02x02_Odd_Even, Connector_PinSocket_2.54mm:PinSocket_1x04_P2.54mm_Vertical, F.Cu at (14.0, 136.9)
- added J25: Conn_01x03, Connector_PinSocket_2.54mm:PinSocket_1x03_P2.54mm_Vertical, F.Cu at (2.54, 136.9)
- added J26: Conn_01x03, Connector_PinSocket_2.54mm:PinSocket_1x03_P2.54mm_Vertical, F.Cu at (28.1, 136.9)
- added JP11: ~OE Low Fixed, Connector_PinHeader_2.54mm:PinHeader_1x02_P2.54mm_Vertical, F.Cu at (24.9, 160.9)
- added JP12: VIA2_CS2, Connector_PinHeader_2.54mm:PinHeader_1x03_P2.54mm_Vertical, F.Cu at (3.17, 120.9)
- added JP13: VIA1_CS1, Connector_PinHeader_2.54mm:PinHeader_1x03_P2.54mm_Vertical, F.Cu at (0.63, 120.9)
- added JP14: A_CS0, Connector_PinHeader_2.54mm:PinHeader_1x03_P2.54mm_Vertical, F.Cu at (5.71, 120.9)
- added JP15: V1_CS1_Select, Connector_PinHeader_2.54mm:PinHeader_1x03_P2.54mm_Vertical, F.Cu at (17.8, 120.9)
- added JP16: V2_CS1_Select, Connector_PinHeader_2.54mm:PinHeader_1x03_P2.54mm_Vertical, F.Cu at (20.4, 120.9)
- added JP17: A_CS0_Select, Connector_PinHeader_2.54mm:PinHeader_1x03_P2.54mm_Vertical, F.Cu at (22.9, 120.9)
- added JP18: V1_CS2_Select, Connector_PinHeader_2.54mm:PinHeader_1x03_P2.54mm_Vertical, F.Cu at (35.0, 120.9)
- added JP19: V2_CS2_Select, Connector_PinHeader_2.54mm:PinHeader_1x03_P2.54mm_Vertical, F.Cu at (37.6, 120.9)
- added JP20: A_CS1_Select, Connector_PinHeader_2.54mm:PinHeader_1x03_P2.54mm_Vertical, F.Cu at (40.1, 120.9)
- moved JP10 12.5 mm to (32.5, 163.4), turned to 180 degrees
- moved C4 10.1 mm to (-9.11, 123.6), turned to 180 degrees
- moved R39 5.52 mm to (24.9, 153.6)
- moved U29 5.50 mm to (4.57, 149.9)
- moved U4 4.82 mm to (-16.6, 127.2)
- moved R4 2.54 mm to (-9.13, 120.2)
- moved J20 2.54 mm to (7.93, 163.4)
- moved C5 2.01 mm to (-5.27, 143.1), turned to 90 degrees
Connections:
- J12 pad 25: ~ROM_OE -> ~RAM_OE
- U11 pad 23: ~IOCS -> ~IOCS_V2
- U11 pad 24: a11 -> Net-(JP12-Pad2)
- U12 pad 23: ~IOCS -> ~IOCS_V1
- U12 pad 24: a12 -> Net-(JP13-Pad2)
- U2 pad 3: ~ROM_OE -> ~RAM_OE
- U2 pad 4: ~ROM_OE -> ~RAM_OE
- U29 pad 19: ~IOCS -> ~IO1
- U29 pad 20: ~ROM -> ~ROM_CS
- U29 pad 21: ~RAM -> ~RAM_CS
- U29 pad 23: ~OE -> ~RAM_OE
- U5 pad 2: a10 -> Net-(JP14-Pad2)
- U5 pad 3: ~IOCS -> ~IOCS_A
- U8 pad 22: ~ROM_OE -> ~RAM_OE
- U9 pad 22: ~RAM_CS -> ~RAM_OE
Routing:
- net +5V: track 222.2 -> 554.8 mm, vias 5 -> 11
- net ~IOCS_V1: track 0.00 -> 275.1 mm, vias 0 -> 3
- net ~RAM_OE: track 0.00 -> 263.2 mm, vias 0 -> 2
- net Net-(JP13-Pad2): track 0.00 -> 237.0 mm, vias 0 -> 2
- net ModIn: track 11.8 -> 239.4 mm, vias 0 -> 1
- net DataOut: track 0.00 -> 189.1 mm
- net ~ROM_CS: track 166.5 -> 304.7 mm, vias 4 -> 6
- net ~RAM_CS: track 141.9 -> 279.3 mm, vias 2 -> 3
- net Net-(JP14-Pad2): track 0.00 -> 121.6 mm, vias 0 -> 2
- net ~ROM_OE: track 119.3 -> 0.00 mm, vias 1 -> 0
- net ~IOCS_A: track 0.00 -> 113.6 mm, vias 0 -> 3
- net ~IOCS: track 324.2 -> 210.9 mm
- net a7: track 361.9 -> 474.7 mm, vias 4 -> 5
- net a6: track 365.8 -> 477.1 mm
- net a8: track 353.3 -> 463.3 mm, vias 3 -> 4
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- removed copper zone on F.Cu, net +5V
- removed copper zone on B.Cu, net GND
Other:
- board text added: "< Axx"
- board text added: "Adjust"
- board text added: "Adjust | Fixed"
- board text added: "Adjustable Address Decoder"
- board text added: "Axx | +5V"
- board text added: "Axx | IOCS"
- board text added: "Fixed"
- board text added: "I0>"
- board text added: "IO Chip Select Mapping"
- board text added: "Low Fixed"
- board text added: "MIn"
- board text added: "MOut"
- board text added: "System Bus Expansion Port #3"
- board text added: "System Bus Expansion Port #4"
- board text added: "a_cs0"
- board text added: "a_iocs"
- board text added: "v1_cs1"
- board text added: "v1_iocs"
- board text added: "v2_cs1"
- board text added: "v2_iocs"
- board text added: "~OE"
- board text removed: "EN | OFF"
- board text removed: "Flexible Address Decoder"
- board text removed: "ModIn"
- board text removed: "ModOut"

Commit message: release revisions
REv001,002 and HEX
Parts:
- added J27: LED SWITCH, Connector_PinHeader_2.54mm:PinHeader_1x03_P2.54mm_Vertical, F.Cu at (210.6, 69.3)
- moved RV3 4.50 mm to (208.0, 81.8)
Connections:
- J12 pad 1: d0 -> db0
- J12 pad 10: a4 -> ab4
- J12 pad 11: d5 -> db5
- J12 pad 12: a5 -> ab5
- J12 pad 13: d6 -> db6
- J12 pad 14: a6 -> ab6
- J12 pad 15: d7 -> db7
- J12 pad 16: a7 -> ab7
- J12 pad 17: a9 -> ab9
- J12 pad 18: a8 -> ab8
- J12 pad 19: a11 -> ab11
- J12 pad 2: a0 -> ab0
- J12 pad 20: a10 -> ab10
- J12 pad 21: a13 -> ab13
- J12 pad 22: a12 -> ab12
- J12 pad 23: a15 -> ab15
- J12 pad 24: a14 -> ab14
- J12 pad 3: d1 -> db1
- J12 pad 4: a1 -> ab1
- J12 pad 5: d2 -> db2
- J12 pad 6: a2 -> ab2
- J12 pad 7: d3 -> db3
- J12 pad 8: a3 -> ab3
- J12 pad 9: d4 -> db4
- RV3 pad 2: LED_bright -> Net-(J27-Pad3)
- U21 pad 12: Net-(U21-Pad12) -> db0
- U21 pad 13: Net-(U21-Pad13) -> db1
- U21 pad 14: Net-(U21-Pad14) -> db2
- U21 pad 15: Net-(U21-Pad15) -> db3
- U21 pad 16: Net-(U21-Pad16) -> db4
- U21 pad 17: Net-(U21-Pad17) -> db5
- U21 pad 18: Net-(U21-Pad18) -> db6
- U21 pad 19: Net-(U21-Pad19) -> db7
- U22 pad 12: Net-(U22-Pad12) -> ab8
- U22 pad 13: Net-(U22-Pad13) -> ab9
- U22 pad 14: Net-(U22-Pad14) -> ab10
- U22 pad 15: Net-(U22-Pad15) -> ab11
- U22 pad 16: Net-(U22-Pad16) -> ab12
- U22 pad 17: Net-(U22-Pad17) -> ab13
- U22 pad 18: Net-(U22-Pad18) -> ab14
- U22 pad 19: Net-(U22-Pad19) -> ab15
- U23 pad 12: Net-(U23-Pad12) -> ab0
- U23 pad 13: Net-(U23-Pad13) -> ab1
- U23 pad 14: Net-(U23-Pad14) -> ab2
- U23 pad 15: Net-(U23-Pad15) -> ab3
- U23 pad 16: Net-(U23-Pad16) -> ab4
- U23 pad 17: Net-(U23-Pad17) -> ab5
- U23 pad 18: Net-(U23-Pad18) -> ab6
- U23 pad 19: Net-(U23-Pad19) -> ab7
- U25 pad 11: Net-(U21-Pad12) -> db0
- U25 pad 12: Net-(U21-Pad13) -> db1
- U25 pad 13: Net-(U21-Pad14) -> db2
- U25 pad 14: Net-(U21-Pad15) -> db3
- U25 pad 17: Net-(U21-Pad16) -> db4
- U25 pad 18: Net-(U21-Pad17) -> db5
- U25 pad 19: Net-(U21-Pad18) -> db6
- U25 pad 20: Net-(U21-Pad19) -> db7
- U26 pad 11: Net-(U22-Pad12) -> ab8
- U26 pad 12: Net-(U22-Pad13) -> ab9
- U26 pad 13: Net-(U22-Pad14) -> ab10
- U26 pad 14: Net-(U22-Pad15) -> ab11
- U26 pad 17: Net-(U22-Pad16) -> ab12
- U26 pad 18: Net-(U22-Pad17) -> ab13
- U26 pad 19: Net-(U22-Pad18) -> ab14
- U26 pad 20: Net-(U22-Pad19) -> ab15
- U27 pad 11: Net-(U23-Pad12) -> ab0
- U27 pad 12: Net-(U23-Pad13) -> ab1
- U27 pad 13: Net-(U23-Pad14) -> ab2
- U27 pad 14: Net-(U23-Pad15) -> ab3
- U27 pad 17: Net-(U23-Pad16) -> ab4
- U27 pad 18: Net-(U23-Pad17) -> ab5
- U27 pad 19: Net-(U23-Pad18) -> ab6
- U27 pad 20: Net-(U23-Pad19) -> ab7
Routing:
- net ab0: track 0.00 -> 161.4 mm, vias 0 -> 1
- net ab1: track 0.00 -> 160.2 mm, vias 0 -> 1
- net ab2: track 0.00 -> 159.7 mm, vias 0 -> 1
- net ab3: track 0.00 -> 159.6 mm, vias 0 -> 1
- net ab6: track 0.00 -> 159.1 mm, vias 0 -> 1
- net ab7: track 0.00 -> 159.0 mm, vias 0 -> 1
- net ab4: track 0.00 -> 159.0 mm, vias 0 -> 1
- net ab5: track 0.00 -> 158.5 mm, vias 0 -> 1
- net Net-(U23-Pad19): track 133.0 -> 0.00 mm
- net Net-(U23-Pad18): track 128.2 -> 0.00 mm
- net Net-(U23-Pad17): track 123.4 -> 0.00 mm
- net ab14: track 0.00 -> 121.5 mm
- net ab15: track 0.00 -> 119.2 mm
- net Net-(U23-Pad16): track 117.8 -> 0.00 mm
- net ab12: track 0.00 -> 116.2 mm
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- added copper zone on F.Cu, net +5V
- added copper zone on B.Cu, net GND
Other:
- board text added: "Board revision: v002"
- board text added: "CS0"
- board text added: "CS1"
- board text added: "I0CS>"
- board text added: "LED OFF | ON"
- board text added: "V1"
- board text added: "V1|V2|A>"
- board text added: "V2"
- board text added: "~NC"
- board text added: "~RAMOE"
- board text removed: "Board revision: v001"
- board text removed: "~ROMOE"
