File: KiCad/Rev003/6502_IO.sch (KiCad schematic (older format))
At the start: 18 parts, among them J11 LCD Connector, J2 Optional UART Port, J33 VIA2PA, J6 Mini-DIN-6, J8 AVR-ISP-10, J9 VIA2PB, U10 ATtiny4313-PU, U11 65C22S, U12 65C22S, U5 65C51N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

Commit message: PDF Schematic Added
Other:
- note added: "Added modem to VIA2 PORT B"
- note added: "Removal of onboard FTDI serial from the DB design"
- note removed: "Added modem to via"
- note removed: "Removal of onboard FTDI serial."
Changed lines of the file:
@@
 v2pa0
 Text Notes 3075 2525 0    50   ~ 0
-Added modem to via
+Added modem to VIA2 PORT B
 Wire Notes Line
 	6275 2575 6675 2575
@@
 	3300 7575 3300 6200
 Text Notes 4150 6900 0    50   ~ 0
- Removal of onboard FTDI serial.
+ Removal of onboard FTDI serial from the DB design
 NoConn ~ 1750 6200
 Wire Wire Line
