File: KiCad/Rev003/AT_65C02_Computer_Rev003.sch (KiCad schematic (older format))
At the start: 36 parts, among them J1 CLK Jumper, J29 Decoder Signals, J7 Expansion port, SW4 SW_SPDT, U1 74HC21, U2 74HC00, U3 74HC02, U4 NE555, U7 65C02S, U8 28C256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

Commit message: U8 ZIF socket
Parts:
- U8: footprint Package_DIP:DIP-28_W15.24mm_Socket -> Socket:DIP_Socket-28_W11.9_W12.7_W15.24_W17.78_W18.5_3M_228-1277-00-0602J
Other:
- note added: "U8 ZIF socket optional\nHEX Expansion board will need\ngreater standoff if ZIF in use"
Changed lines of the file:
@@
 Sheet 1 7
 Title "AT65C02 Hobby Computer"
-Date "2023-04-05"
+Date "2023-05-01"
 Rev "Rev003"
 Comp "This AT65C02 version by AdamT117. "
@@
 F 0 "U8" H 1550 5915 50  0000 C CNN
 F 1 "28C256" H 1550 5824 50  0000 C CNN
-F 2 "Package_DIP:DIP-28_W15.24mm_Socket" H 1500 5800 50  0001 C CNN
+F 2 "Socket:DIP_Socket-28_W11.9_W12.7_W15.24_W17.78_W18.5_3M_228-1277-00-0602J" H 1500 5800 50  0001 C CNN
 F 3 "http://ww1.microchip.com/downloads/en/DeviceDoc/doc0006.pdf" H 1550 5000 50  0001 C CNN
 	1    1550 5000
@@
 Text Notes 550  3075 0    50   ~ 0
 Breakout all CPU pins to headers\nDefault:NMI and RDY \ndefault tied High
-Text Notes 1800 3825 0    50   ~ 0
+Text Notes 2225 3775 0    50   ~ 0
 RAM and ROM OE CS seperated for adjustable decoder option.\nROM WE breakout for onboard ROM programming
 Text Notes 8350 5150 0    50   ~ 0
@@
 Wire Bus Line
 	5350 4250 5350 5750
+Text Notes 700  3950 0    50   ~ 0
+U8 ZIF socket optional\nHEX Expansion board will need\ngreater standoff if ZIF in use
 $EndSCHEMATC

Commit message: Update AT_65C02_Computer_Rev003.sch
Other:
- note added: "CLK"
- note added: "ROM~OE"
- note added: "a15"
Changed lines of the file:
@@
 Text Notes 3800 3275 0    50   ~ 0
 Breakout all CPU pins to headers\nDefault:BE and ~SO~ default tied High
+Text Notes 700  3950 0    50   ~ 0
+U8 ZIF socket optional\nHEX Expansion board will need\ngreater standoff if ZIF in use
 Wire Bus Line
 	3100 5450 3100 5650
@@
 Wire Bus Line
 	5350 4250 5350 5750
-Text Notes 700  3950 0    50   ~ 0
-U8 ZIF socket optional\nHEX Expansion board will need\ngreater standoff if ZIF in use
+Text Notes 5875 1100 0    50   ~ 0
+ROM~OE
+Text Notes 4725 1300 0    50   ~ 0
+a15
+Text Notes 5525 1700 0    50   ~ 0
+CLK
 $EndSCHEMATC
