File: KiCad/Rev003/Power_Connectors.sch (KiCad schematic (older format))
At the start: 15 parts, among them J12 System Bus Output port, J14 ESP Interface, J15 Level_Shifter_HV, J16 Level_Shifter_LV, J18 CPU Signals, J21 Expansion port #2, J22 Expansion port #3, J5 Barrel_Jack-Connector, SW1 SW_SPDT, U13 LM3940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

Commit message: PDF Schematic Added
Other:
- note added: "Added header for the additional signals\nfrom CPU and ROM"
- note added: "Level shifter and ESP port"
- note removed: "Added header for the additional signals\nCPU and ROM"
- note removed: "Level shifter and ESP pin order may need adjustment to suit layout\n** Note Level shifter mirror error to correct"
Changed lines of the file:
@@
 Port is via blinky latches for display expansion (HEX board)
 Text Notes 2400 2475 0    50   ~ 0
-Level shifter and ESP pin order may need adjustment to suit layout\n** Note Level shifter mirror error to correct
+Level shifter and ESP port
 Text Notes 6650 2775 0    50   ~ 0
 L7805\nCurrent consumption with full blinky \nand HEX display @0.4amps\n\nTemperature 60 degrees C
@@
 	8975 4775 9225 4775
 Text Notes 8575 5325 0    50   ~ 0
-Added header for the additional signals\nCPU and ROM
+Added header for the additional signals\nfrom CPU and ROM
 Wire Notes Line
 	9825 3375 10350 3375
@@
 Wire Wire Line
 	9450 3300 9450 3400
+Connection ~ 9450 3300
 Wire Bus Line
 	2775 5225 2775 6150
@@
 Wire Bus Line
 	750  6100 750  7650
-Connection ~ 9450 3300
 $EndSCHEMATC
