File: KiCad/Hex Display Rev002/AT65C02_HEX_rev002.sch (KiCad schematic (older format))
At the start: 43 parts, among them J1 Expansion Connector, J2 Conn_02x03_Odd_Even, J3 Conn_01x03, Q1 BC557, Q2 BC557, Q3 BC557, Q4 BC557, Q5 BC557, Q6 BC557, U1 NE555P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

Commit message: Images added
Connections:
- net GND: no longer J1.30 (Pin_30), J2.5 (Pin_5)
- net RAM_~OE~: now reaches J1.27 (Pin_27)
- net RAM_~OE~: now also J2.4 (Pin_4)
- net +3.3V renamed ~IRQ
- net ~RAM_CS renamed RAM_~CS
- net ~ROM_CS renamed ROM_~CS
- net ~ROM_OE renamed ROM_~OE
- new net R~W: J1.30 (Pin_30), J2.5 (Pin_5)
- no-connect marks 21 -> 19
Other:
- note added: "Expansion Port revised to match Rev003 board"
- note added: "Multiplexer Clock"
- moved on the sheet: C1, C2, C3, C4, C5, J1, J2, J3, Q1, Q2, Q3, Q4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
