File: KiCad/Hex Display Rev002/AT65c02_HEX_rev002.kicad_pcb (KiCad board)
At the start: 2 copper layers, 86.9 x 83.1 mm, 48 parts, among them J1 Expansion Connector, J2 Conn_02x03_Odd_Even, J3 Conn_01x03, Q1 BC557, Q2 BC557, Q3 BC557, Q4 BC557, Q5 BC557, Q6 BC557, U1 NE555P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

Commit message: Images added
Parts:
- removed ?: , 
- removed REF**: MountingHole_2.1mm, MountingHole:MountingHole_2.1mm
- removed REF**: MountingHole_2.5mm, MountingHole:MountingHole_2.5mm
- removed REF**: KiCad-Logo2_8mm_SilkScreen, Symbol:KiCad-Logo2_8mm_SilkScreen
- removed REF**: OSHW-Logo_11.4x12mm_SilkScreen, Symbol:OSHW-Logo_11.4x12mm_SilkScreen
Connections:
- net +3.3V renamed ~IRQ
- net ~RAM_CS renamed RAM_~CS
- net ~ROM_CS renamed ROM_~CS
- net ~ROM_OE renamed ROM_~OE
- J1 pad 27: Net-(J1-Pad27) -> RAM_~OE~
- J1 pad 30: GND -> R~W
- J2 pad 4: Net-(J2-Pad4) -> RAM_~OE~
- J2 pad 5: GND -> R~W
Routing:
- net R~W: track 0.00 -> 13.0 mm
- net RAM_~OE~: track 0.00 -> 12.9 mm
- net GND: track 124.2 -> 115.4 mm
Other:
- board text added: "Board revision: v002"
- board text added: "R~W RAM~CS~ ROM~CS~"
- board text added: "~IRQ RAM~OE~ ROM~OE~"
- board text removed: "+3.3V NC ~ROMOE"
- board text removed: "Board revision: v001"
- board text removed: "GND ~RAMCS ~ROMCS"
