File: KiCad/Memory Decoder/Memory Decoder.sch (KiCad schematic (older format))
At the start: 11 parts, among them J1 IOCS/Decoder Signals Expansio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, J2 Conn_02x02_Odd_Even, J3 Decoder Signals, J4 Conn_02x03_Odd_Even, J5 Memory Decoder Expansion, J6 ~IOx, J7 ~IRQx, SW1 SW_DIP_x04, SW2 SW_DIP_x04, U1 Flexible Memory Decoder

Commit message: Gerbers Added
Parts:
- C1: symbol 65C02_Computer-rescue:C-Device -> Memory-Decoder-rescue:C-Device-65C02_Computer-rescue
Changed lines of the file:
@@
 $Descr A4 11693 8268
 encoding utf-8
-Sheet 1 2
-Title ""
-Date ""
-Rev ""
-Comp ""
+Sheet 1 1
+Title "AT65C02 Programmable Memory Decoder"
+Date "2023-04-05"
+Rev "Rev001"
+Comp "by AdamT117"
 Comment1 ""
 Comment2 ""
 Comment3 ""
-Comment4 ""
+Comment4 "Expansion board for AT65C02"
 $EndDescr
 Text GLabel 1100 950  0    50   Input ~ 0
@@
 	-1   0    0    -1
 $EndComp
-$Sheet
-S 10325 675  500  150
-U 647F3D88
-F0 "Sheet647F3D87" 50
-F1 "file647F3D87.sch" 50
-$EndSheet
 Text Label 2150 3275 2    50   ~ 0
 a15
@@
 	9000 3200 6725 3200
 $Comp
-L 65C02_Computer-rescue:GND-power #PWR?
+L Memory-Decoder-rescue:GND-power-65C02_Computer-rescue #PWR?
 U 1 1 64860E97
 P 7800 2825
@@
 $EndComp
 $Comp
-L 65C02_Computer-rescue:+5V-power #PWR?
+L Memory-Decoder-rescue:+5V-power-65C02_Computer-rescue #PWR?
 U 1 1 64860E9D
 P 7800 1225
@@
 	8700 1200 8700 1425
 $Comp
-L 65C02_Computer-rescue:+5V-power #PWR?
+L Memory-Decoder-rescue:+5V-power-65C02_Computer-rescue #PWR?
 U 1 1 641E664E
 P 3425 4425
@@
 	950  7525 950  7575
 $Comp
-L 65C02_Computer-rescue:C-Device C?
+L Memory-Decoder-rescue:C-Device-65C02_Computer-rescue C?
 U 1 1 641CA3DF
 P 950 7375
@@
 $EndComp
 $Comp
-L 65C02_Computer-rescue:+5V-power #PWR?
+L Memory-Decoder-rescue:+5V-power-65C02_Computer-rescue #PWR0104
 U 1 1 641CA3E5
 P 950 7125
-F 0 "#PWR?" H 950 6975 50  0001 C CNN
+F 0 "#PWR0104" H 950 6975 50  0001 C CNN
 F 1 "+5V" H 965 7298 50  0000 C CNN
 F 2 "" H 950 7125 50  0001 C CNN
