File: KiCad/Debugger/debugger/debugger.kicad_pcb (KiCad board)
At the start: 2 copper layers, 65.5 x 84.8 mm, 12 parts, among them J1 Conn_02x16_Odd_Even, J2 Conn_02x16_Odd_Even, J3 CPU Signals, J4 Conn_02x18_Odd_Even, SW4 SW_SPDT

Commit message: debugger wip
Parts:
- removed the REF** at (114.8, 96.1)
- removed the REF** at (91.9, 91.2)
- removed the REF** at (140.2, 96.2)
- removed the REF** at (91.9, 114.0)
- removed the REF** at (140.2, 73.4)
- removed the REF** at (140.2, 118.1)
- removed the REF** at (91.9, 68.3)
- removed SW4: SW_SPDT, Button_Switch_THT:SW_PUSH_6mm
- added J10: Conn_01x08, Connector_PinSocket_2.54mm:PinSocket_1x08_P2.54mm_Vertical, F.Cu at (71.3, -12.1)
- added J11: Conn_01x08, Connector_PinHeader_2.54mm:PinHeader_1x08_P2.54mm_Vertical, F.Cu at (58.6, 28.5)
- added J12: Conn_01x08, Connector_PinHeader_2.54mm:PinHeader_1x08_P2.54mm_Vertical, B.Cu at (76.3, -14.7)
- added J13: Conn_01x08, Connector_PinHeader_2.54mm:PinHeader_1x08_P2.54mm_Vertical, B.Cu at (71.3, -14.7)
- added J14: Conn_01x08, Connector_PinHeader_2.54mm:PinHeader_1x08_P2.54mm_Vertical, B.Cu at (99.2, 33.6)
- added J15: Conn_01x10, Connector_PinHeader_2.54mm:PinHeader_1x10_P2.54mm_Vertical, F.Cu at (49.4, -9.58)
- added J16: Conn_01x10, Connector_PinSocket_2.54mm:PinSocket_1x10_P2.54mm_Vertical, F.Cu at (49.4, -12.1)
- added J17: Conn_01x10, Connector_PinHeader_2.54mm:PinHeader_1x10_P2.54mm_Vertical, B.Cu at (49.4, -14.7)
- added J18: Conn_01x08, Connector_PinHeader_2.54mm:PinHeader_1x08_P2.54mm_Vertical, B.Cu at (53.5, 33.6)
- added J19: Conn_01x08, Connector_PinSocket_2.54mm:PinSocket_1x08_P2.54mm_Vertical, F.Cu at (53.5, 31.1)
- added J20: Conn_01x08, Connector_PinHeader_2.54mm:PinHeader_1x08_P2.54mm_Vertical, F.Cu at (35.7, 28.5)
- added J21: Conn_02x18_Odd_Even, Connector_PinHeader_2.54mm:PinHeader_2x18_P2.54mm_Vertical, F.Cu at (112.5, -14.7)
- added J5: Conn_01x08, Connector_PinHeader_2.54mm:PinHeader_1x08_P2.54mm_Vertical, F.Cu at (71.3, -9.58)
- added J6: Conn_01x08, Connector_PinHeader_2.54mm:PinHeader_1x08_P2.54mm_Vertical, F.Cu at (76.3, -9.58)
- added J7: Conn_01x08, Connector_PinSocket_2.54mm:PinSocket_1x08_P2.54mm_Vertical, F.Cu at (58.6, 31.1)
- added J8: Conn_01x08, Connector_PinSocket_2.54mm:PinSocket_1x08_P2.54mm_Vertical, F.Cu at (76.3, -12.1)
- added J9: Conn_01x08, Connector_PinSocket_2.54mm:PinSocket_1x08_P2.54mm_Vertical, F.Cu at (99.2, 31.1)
- added REF**: OSHW-Logo2_7.3x6mm_SilkScreen, Symbol:OSHW-Logo2_7.3x6mm_SilkScreen, F.Cu at (29.7, 31.6)
- added XA1: Arduino_Mega2560_Shield, PCM_arduino-library:Arduino_Mega2560_Shield, F.Cu at (7.77, 36.1)
- J1: value Conn_02x16_Odd_Even -> Conn_02x18_Odd_Even; footprint Connector_PinHeader_2.54mm:PinHeader_2x16_P2.54mm_Vertical -> Connector_PinHeader_2.54mm:PinHeader_2x18_P2.54mm_Vertical
- J2: value Conn_02x16_Odd_Even -> Conn_02x20_Odd_Even; footprint Connector_PinHeader_2.54mm:PinHeader_2x16_P2.54mm_Vertical -> Connector_IDC:IDC-Header_2x20_P2.54mm_Vertical; moved to F.Cu
- J3: value CPU Signals -> Conn_01x08; footprint Connector_PinHeader_2.54mm:PinHeader_2x06_P2.54mm_Vertical -> Connector_PinHeader_2.54mm:PinHeader_1x08_P2.54mm_Vertical
- J4: value Conn_02x18_Odd_Even -> Conn_01x08; footprint Connector_PinHeader_2.54mm:PinHeader_2x18_P2.54mm_Vertical -> Connector_PinHeader_2.54mm:PinHeader_1x08_P2.54mm_Vertical
- moved J2 110.4 mm to (40.8, 18.4), turned to 90 degrees
- moved J1 98.4 mm to (104.3, -14.7)
- moved J3 74.5 mm to (58.6, 33.6)
- moved J4 68.2 mm to (81.4, 28.5), turned to 90 degrees
Connections:
- J1 pad 1: /a0 -> ~{RES}
- J1 pad 10: /d4 -> SYNC
- J1 pad 11: /a5 -> /d0
- J1 pad 12: /d5 -> /a0
- J1 pad 13: /a6 -> /d1
- J1 pad 14: /d6 -> /a1
- J1 pad 15: /a7 -> /d2
- J1 pad 16: /d7 -> /a2
- J1 pad 17: /a8 -> /d3
- J1 pad 18: CLK -> /a3
- J1 pad 19: /a9 -> /d4
- J1 pad 2: /d0 -> unconnected-(J1-Pin_2-Pad2)
- J1 pad 20: R~{W} -> /a4
- J1 pad 21: /a10 -> /d5
- J1 pad 22: ~{IOCS} -> /a5
- J1 pad 23: /a11 -> /d6
- J1 pad 24: ~{RES} -> /a6
- J1 pad 25: /a12 -> /d7
- J1 pad 26: ~{IRQX} -> /a7
- J1 pad 27: /a13 -> /a15
- J1 pad 28: unconnected-(J1-Pin_28-Pad28) -> /a8
- J1 pad 3: /a1 -> ~{SO}
- J1 pad 30: GND -> /a9
- J1 pad 31: /a15 -> /a13
- J1 pad 32: +5V -> /a10
- J1 pad 4: /d1 -> RDY
- J1 pad 5: /a2 -> ~{BE}
- J1 pad 6: /d2 -> ~{IRQ}
- J1 pad 7: /a3 -> R~{W}
- J1 pad 8: /d3 -> ~{NMI}
- J1 pad 9: /a4 -> unconnected-(J1-Pin_9-Pad9)
- J2 pad 1: /a0 -> ~{RES}
- J2 pad 10: /d4 -> /a0
- J2 pad 11: /a5 -> /d0
- J2 pad 12: /d5 -> /a1
- J2 pad 13: /a6 -> /d1
- J2 pad 14: /d6 -> /a2
- J2 pad 15: /a7 -> /d2
- J2 pad 16: /d7 -> /a3
- J2 pad 17: /a8 -> /d3
- J2 pad 18: CLK -> /a4
- J2 pad 19: /a9 -> /d4
- J2 pad 2: /d0 -> RDY
- J2 pad 20: R~{W} -> /a5
- J2 pad 21: /a10 -> /d5
- J2 pad 22: ~{IOCS} -> /a6
- J2 pad 23: /a11 -> /d6
- J2 pad 24: ~{RES} -> /a7
- J2 pad 25: /a12 -> /d7
- J2 pad 26: ~{IRQX} -> /a8
- J2 pad 27: /a13 -> /a15
- J2 pad 28: unconnected-(J2-Pin_28-Pad28) -> /a9
- J2 pad 3: /a1 -> ~{SO}
- J2 pad 30: GND -> /a10
- J2 pad 31: /a15 -> /a13
- J2 pad 32: +5V -> /a11
- J2 pad 4: /d1 -> ~{IRQ}
- J2 pad 5: /a2 -> ~{BE}
- J2 pad 6: /d2 -> ~{NMI}
- J2 pad 7: /a3 -> R~{W}
- J2 pad 8: /d3 -> SYNC
- J2 pad 9: /a4 -> unconnected-(J2-Pin_9-Pad9)
- J3 pad 1: ~{VP} -> Net-(J11-Pin_1)
- J3 pad 2: RDY -> Net-(J11-Pin_2)
- J3 pad 3: ~{NMI} -> Net-(J11-Pin_3)
- J3 pad 4: PHI1O -> Net-(J11-Pin_4)
- J3 pad 5: ~{IRQ} -> Net-(J11-Pin_5)
- J3 pad 6: ~{ML} -> Net-(J11-Pin_6)
- J3 pad 7: PHI2O -> Net-(J11-Pin_7)
- J3 pad 8: SYNC -> Net-(J11-Pin_8)
- J4 pad 1: unconnected-(J4-Pin_1-Pad1) -> Net-(J14-Pin_8)
- J4 pad 2: ~{RES} -> Net-(J14-Pin_7)
- J4 pad 3: RDY -> Net-(J14-Pin_6)
- J4 pad 4: ~{SO} -> Net-(J14-Pin_5)
- J4 pad 5: ~{IRQ} -> Net-(J14-Pin_4)
- J4 pad 6: ~{BE} -> Net-(J14-Pin_3)
- J4 pad 7: ~{NMI} -> Net-(J14-Pin_2)
- J4 pad 8: R~{W} -> Net-(J14-Pin_1)
Routing:
- net /a15: track 71.8 -> 0.00 mm
- net ~{RES}: track 67.3 -> 0.00 mm
- net /a14: track 63.0 -> 0.00 mm
- net R~{W}: track 60.7 -> 0.00 mm
- net /a13: track 54.9 -> 0.00 mm
- net RDY: track 29.7 -> 83.7 mm
- net /a11: track 53.5 -> 0.00 mm
- net /a12: track 53.4 -> 0.00 mm
- net /a10: track 50.7 -> 0.00 mm
- net /a9: track 48.2 -> 0.00 mm
- net /a8: track 46.5 -> 0.00 mm
- net /a7: track 44.7 -> 0.00 mm
- net /a6: track 43.0 -> 0.00 mm
- net /a5: track 41.2 -> 0.00 mm
- net /a4: track 39.4 -> 0.00 mm
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Other:
- board size 65.5 x 84.8 mm -> 97 x 53.3 mm
- board text added: "3V3"
- board text added: "5V3"
- board text added: "5V4"
- board text added: "A0"
- board text added: "A1"
- board text added: "A10"
- board text added: "A11"
- board text added: "A12"
- board text added: "A13"
- board text added: "A14"
- board text added: "A15"
- board text added: "A2"
- board text added: "A3"
- board text added: "A4"
- board text added: "A5"
- board text added: "A6"
- board text added: "A7"
- board text added: "A8"
- board text added: "A9"
- board text added: "AREF"
- board text added: "AT65C02 Diagnostic Tool"
- board text added: "AT65C02 HEADER"
- board text added: "Arduino Mega Shield"
- board text added: "D0"
- board text added: "D1"
- board text added: "D10"
- board text added: "D11"
- board text added: "D12"
- board text added: "D13"
- board text added: "D14"
- board text added: "D15"
- board text added: "D16"
- board text added: "D17"
- board text added: "D18"
- board text added: "D19"
- board text added: "D2"
- board text added: "D20"
- board text added: "D21"
- board text added: "D22"
- board text added: "D23"
- board text added: "D24"
- board text added: "D25"
- board text added: "D26"
- board text added: "D27"
- board text added: "D28"
- board text added: "D29"
- board text added: "D3"
- board text added: "D30"
- board text added: "D31"
- board text added: "D32"
- board text added: "D33"
- board text added: "D34"
- board text added: "D35"
- board text added: "D36"
- board text added: "D37"
- board text added: "D38"
- board text added: "D39"
- board text added: "D4"
- board text added: "D40"
- board text added: "D41"
- board text added: "D42"
- board text added: "D43"
- board text added: "D44"
- board text added: "D45"
- board text added: "D46"
- board text added: "D47"
- board text added: "D48"
- board text added: "D49"
- board text added: "D5"
- board text added: "D6"
- board text added: "D7"
- board text added: "D8"
- board text added: "D9"
- board text added: "GND1"
- board text added: "GND2"
- board text added: "GND3"
- board text added: "GND5"
- board text added: "GND6"
- board text added: "ICSP"
- board text added: "IREF"
- board text added: "Interactive Diagnostic Tool by Nectivio"
- board text added: "MISO"
- board text added: "MOSI"
- board text added: "NC"
- board text added: "RST"
- board text added: "SCK"
- board text added: "SCL"
- board text added: "SDA"
- board text added: "SS"
- board text added: "VIN"
- board text removed: "locked"
