File: KiCad/Hex Display Rev003/AT65C02_HEX_rev003.kicad_pcb (KiCad board)
At the start: 2 copper layers, 86.9 x 83.1 mm, 45 parts, among them J1 Expansion Connector, J3 Conn_01x03, Q1 BC557, Q2 BC557, Q3 BC557, Q4 BC557, Q5 BC557, Q6 BC557, U1 NE555P, U10 E10561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

Commit message: Rev004 revisions
Other:
- board text added: "Board revision: v003"
- board text removed: "Board revision: v002"

Commit message: Hex board Resistor value update
Parts:
- R10, R13, R14, R9: value 4k7 -> 18k
- R17: value 4k7 -> 680
- R18: value 2k2 -> 680
Other:
- board text added: "18k"
- board text added: "2k2"
- board text added: "680"
