File: KiCad/Hex Display Rev003/AT65C02_HEX_rev003.sch (KiCad schematic (older format))
At the start: 43 parts, among them J1 Expansion Connector, J2 Conn_02x03_Odd_Even, J3 Conn_01x03, Q1 BC557, Q2 BC557, Q3 BC557, Q4 BC557, Q5 BC557, Q6 BC557, U1 NE555P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

Commit message: HEX board Rev003
Parts:
- removed J2: Conn_02x03_Odd_Even, Connector_PinSocket_2.54mm:PinSocket_2x03_P2.54mm_Vertical, symbol Connector_Generic:Conn_02x03_Odd_Even
- added H1: MountingHole, MountingHole:MountingHole_2.2mm_M2, symbol Mechanical:MountingHole
- J1: footprint Connector_PinHeader_2.54mm:PinHeader_2x16_P2.54mm_Vertical -> Connector_PinHeader_2.54mm:PinHeader_2x13_P2.54mm_Vertical; symbol Connector_Generic:Conn_02x16_Odd_Even -> Connector_Generic:Conn_02x13_Odd_Even
Connections:
- net labels removed: RAM_~CS, RAM_~OE~, ROM_~CS, ROM_~OE, R~W, ~IRQ
Other:
- note added: "Rev3 - breakouts removed\nROM~CS~, ROM~OE~\nRAM~CS~,RAM~OE\nR~W~,~IRQ~"
Changed lines of the file:
@@
 Sheet 1 1
 Title "AT65C02 HEX Expansion Board"
-Date "2023-04-02"
-Rev "Rev002"
+Date "2023-05-09"
+Rev "Rev003"
 Comp "by AdamT117"
 Comment1 ""
@@
 	1    0    0    -1
 $EndComp
-$Comp
-L Connector_Generic:Conn_02x03_Odd_Even J2
-U 1 1 63F09274
-P 8075 10075
-F 0 "J2" H 8125 10392 50  0000 C CNN
-F 1 "Conn_02x03_Odd_Even" H 8125 10301 50  0000 C CNN
-F 2 "Connector_PinSocket_2.54mm:PinSocket_2x03_P2.54mm_Vertical" H 8075 10075 50  0001 C CNN
-F 3 "~" H 8075 10075 50  0001 C CNN
-	1    8075 10075
-	1    0    0    -1
-$EndComp
-Text GLabel 8375 9975 2    50   Input ~ 0
-ROM_~OE
-Text GLabel 7875 10075 0    50   Input ~ 0
-RAM_~CS
-Text GLabel 7875 9975 0    50   Input ~ 0
-ROM_~CS
-Text GLabel 8375 10175 2    50   Input ~ 0
-~IRQ
 $Comp
 L power:GND #PWR?
@@
 a8
 $Comp
-L Connector_Generic:Conn_02x16_Odd_Even J1
+L Connector_Generic:Conn_02x13_Odd_Even J1
 U 1 1 636992C7
-P 14050 4775
-F 0 "J1" H 14100 5725 50  0000 C CNN
-F 1 "Expansion Connector" H 14100 5650 50  0000 C CNN
-F 2 "Connector_PinHeader_2.54mm:PinHeader_2x16_P2.54mm_Vertical" H 14050 4775 50  0001 C CNN
-F 3 "~" H 14050 4775 50  0001 C CNN
-	1    14050 4775
+P 14050 4675
+F 0 "J1" H 14100 5625 50  0000 C CNN
+F 1 "Expansion Connector" H 14100 5550 50  0000 C CNN
+F 2 "Connector_PinHeader_2.54mm:PinHeader_2x13_P2.54mm_Vertical" H 14050 4675 50  0001 C CNN
+F 3 "~" H 14050 4675 50  0001 C CNN
+	1    14050 4675
 	-1   0    0    -1
 $EndComp
@@
 	14250 5175 14700 5175
 Wire Wire Line
-	14250 5575 14950 5575
-Wire Wire Line
-	13300 5575 13750 5575
+	13300 5275 13750 5275
 $Comp
 L power:GND #PWR0110
 U 1 1 63EE1303
-P 13300 5575
-F 0 "#PWR0110" H 13300 5325 50  0001 C CNN
-F 1 "GND" H 13305 5402 50  0000 C CNN
-F 2 "" H 13300 5575 50  0001 C CNN
-F 3 "" H 13300 5575 50  0001 C CNN
-	1    13300 5575
+P 13300 5275
+F 0 "#PWR0110" H 13300 5025 50  0001 C CNN
+F 1 "GND" H 13305 5102 50  0000 C CNN
+F 2 "" H 13300 5275 50  0001 C CNN
+F 3 "" H 13300 5275 50  0001 C CNN
+	1    13300 5275
 	1    0    0    -1
 $EndComp
@@
 	1    0    0    -1
 $EndComp
-Text GLabel 14250 5475 2    50   Output ~ 0
-~IRQ
-Text GLabel 14250 5275 2    50   Output ~ 0
-ROM_~OE
-Text GLabel 13750 5275 0    50   Output ~ 0
-ROM_~CS
-Text GLabel 13750 5375 0    50   Output ~ 0
-RAM_~CS
 $Comp
 L Connector_Generic:Conn_01x03 J3
@@
 	15425 5575 15425 5475
 NoConn ~ 15150 5175
-Wire Wire Line
-	14950 5175 14950 5575
 Wire Wire Line
 	5675 2600 5675 3225
@@
 Wire Wire Line
 	7225 850  8625 850
-Text GLabel 13750 5475 0    50   Output ~ 0
-R~W
-Text GLabel 14250 5375 2    50   Output ~ 0
-RAM_~OE~
-Text GLabel 7875 10175 0    50   Input ~ 0
-R~W
-Text GLabel 8375 10075 2    50   Input ~ 0
-RAM_~OE~
+Wire Notes Line
+	9000 9600 9000 10525
+Wire Notes Line
+	9000 10525 7325 10525
+Wire Notes Line
+	7325 10525 7325 9600
+Wire Notes Line
+	7325 9600 9000 9600
+Text Notes 9225 10175 0    50   ~ 0
+Rev3 - breakouts removed\nROM~CS~, ROM~OE~\nRAM~CS~,RAM~OE\nR~W~,~IRQ~
+Text Notes 14750 6325 0    50   ~ 0
+Rev3 - breakouts removed\nROM~CS~, ROM~OE~\nRAM~CS~,RAM~OE\nR~W~,~IRQ~
+Wire Wire Line
+	14250 5275 14950 5275
+Wire Wire Line
+	14950 5175 14950 5275
+$Comp
+L Mechanical:MountingHole H1
+U 1 1 646F5389
+P 13725 1300
+F 0 "H1" H 13825 1346 50  0000 L CNN
+F 1 "MountingHole" H 13825 1255 50  0000 L CNN
+F 2 "MountingHole:MountingHole_2.2mm_M2" H 13725 1300 50  0001 C CNN
+F 3 "~" H 13725 1300 50  0001 C CNN
+	1    13725 1300
+	1    0    0    -1
+$EndComp
 Wire Bus Line
 	14800 4775 14800 5800

Commit message: Hex board Resistor value update
Parts:
- R10, R13, R14, R9: value 4k7 -> 18k
- R17: value 4k7 -> 680
- R18: value 2k2 -> 680
Changed lines of the file:
@@
 AR Path="/638AF04F" Ref="R10"  Part="1"
 F 0 "R10" V 8450 5575 50  0000 C CNN
-F 1 "4k7" V 8525 5575 50  0000 C CNN
+F 1 "18k" V 8525 5575 50  0000 C CNN
 F 2 "Resistor_THT:R_Axial_DIN0207_L6.3mm_D2.5mm_P7.62mm_Horizontal" V 8455 5575 50  0001 C CNN
 F 3 "~" H 8525 5575 50  0001 C CNN
@@
 AR Path="/638AF066" Ref="R9"  Part="1"
 F 0 "R9" V 8450 4850 50  0000 C CNN
-F 1 "4k7" V 8525 4850 50  0000 C CNN
+F 1 "18k" V 8525 4850 50  0000 C CNN
 F 2 "Resistor_THT:R_Axial_DIN0207_L6.3mm_D2.5mm_P7.62mm_Horizontal" V 8455 4850 50  0001 C CNN
 F 3 "~" H 8525 4850 50  0001 C CNN
@@
 AR Path="/63D4564B" Ref="R14"  Part="1"
 F 0 "R14" V 8450 7125 50  0000 C CNN
-F 1 "4k7" V 8525 7125 50  0000 C CNN
+F 1 "18k" V 8525 7125 50  0000 C CNN
 F 2 "Resistor_THT:R_Axial_DIN0207_L6.3mm_D2.5mm_P7.62mm_Horizontal" V 8455 7125 50  0001 C CNN
 F 3 "~" H 8525 7125 50  0001 C CNN
@@
 AR Path="/63D45662" Ref="R13"  Part="1"
 F 0 "R13" V 8450 6425 50  0000 C CNN
-F 1 "4k7" V 8525 6425 50  0000 C CNN
+F 1 "18k" V 8525 6425 50  0000 C CNN
 F 2 "Resistor_THT:R_Axial_DIN0207_L6.3mm_D2.5mm_P7.62mm_Horizontal" V 8455 6425 50  0001 C CNN
 F 3 "~" H 8525 6425 50  0001 C CNN
@@
 AR Path="/6384D091" Ref="R18"  Part="1"
 F 0 "R18" V 6575 1325 50  0000 C CNN
-F 1 "2k2" V 6650 1325 50  0000 C CNN
+F 1 "680" V 6650 1325 50  0000 C CNN
 F 2 "Resistor_THT:R_Axial_DIN0207_L6.3mm_D2.5mm_P7.62mm_Horizontal" V 6580 1325 50  0001 C CNN
 F 3 "~" H 6650 1325 50  0001 C CNN
@@
 AR Path="/6384D0A0" Ref="R17"  Part="1"
 F 0 "R17" V 5025 1325 50  0000 C CNN
-F 1 "4k7" V 5100 1325 50  0000 C CNN
+F 1 "680" V 5100 1325 50  0000 C CNN
 F 2 "Resistor_THT:R_Axial_DIN0207_L6.3mm_D2.5mm_P7.62mm_Horizontal" V 5030 1325 50  0001 C CNN
 F 3 "~" H 5100 1325 50  0001 C CNN

Commit message: Refresh 2025
No changes just a refresh and update to readme.
Parts:
- U10, U5, U6, U7, U8, U9: symbol Display_Character:LuckyLight_KWI-561AVB -> AT65C02_HEX_rev003-rescue:LuckyLight_KWI-561AVB-Display_Character
Changed lines of the file:
@@
 	6525 5500 6600 5500
 $Comp
-L Display_Character:LuckyLight_KWI-561AVB U?
+L AT65C02_HEX_rev003-rescue:LuckyLight_KWI-561AVB-Display_Character U?
 U 1 1 638AF080
 P 4925 5100
@@
 $EndComp
 $Comp
-L Display_Character:LuckyLight_KWI-561AVB U?
+L AT65C02_HEX_rev003-rescue:LuckyLight_KWI-561AVB-Display_Character U?
 U 1 1 638AF08A
 P 6225 5100
@@
 	6500 7775 6575 7775
 $Comp
-L Display_Character:LuckyLight_KWI-561AVB U?
+L AT65C02_HEX_rev003-rescue:LuckyLight_KWI-561AVB-Display_Character U?
 U 1 1 64070BE8
 P 4900 7375
@@
 $EndComp
 $Comp
-L Display_Character:LuckyLight_KWI-561AVB U?
+L AT65C02_HEX_rev003-rescue:LuckyLight_KWI-561AVB-Display_Character U?
 U 1 1 64070BF2
 P 6200 7375
@@
 $EndComp
 $Comp
-L Display_Character:LuckyLight_KWI-561AVB U?
+L AT65C02_HEX_rev003-rescue:LuckyLight_KWI-561AVB-Display_Character U?
 U 1 1 6384D0C2
 P 5300 2200
@@
 $EndComp
 $Comp
-L Display_Character:LuckyLight_KWI-561AVB U?
+L AT65C02_HEX_rev003-rescue:LuckyLight_KWI-561AVB-Display_Character U?
 U 1 1 6384D0C8
 P 6725 2200
