File: KiCad/Rev004/6502_IO.sch (KiCad schematic (older format))
At the start: 18 parts, among them J11 LCD Connector, J2 Optional UART Port, J33 VIA2PA, J6 Mini-DIN-6, J8 AVR-ISP-10, J9 VIA2PB, U10 ATtiny4313-PU, U11 65C22S, U12 65C22S, U5 65C51N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

Commit message: minor PCB revisions
Connections:
- net ~CTS: now also J2.1 (Pin_1); no longer J2.5 (Pin_5)
- net ~RTS: now also J2.5 (Pin_5); no longer J2.1 (Pin_1)
Other:
- note added: "08/2023\nCTS RTS swapped to better match my FTDI"
Changed lines of the file:
@@
 Sheet 6 7
 Title "AT65C02 Hobby Computer"
-Date "2023-05-09"
+Date "2023-08-06"
 Rev "Rev004"
 Comp "This AT65C02 version by AdamT117. "
@@
 Text GLabel 1750 6000 0    50   Input ~ 0
 TxD
+Text GLabel 1550 6300 0    50   BiDi ~ 0
+~RTS
 Text GLabel 1575 5900 0    50   BiDi ~ 0
-~RTS
-Text GLabel 1550 6300 0    50   BiDi ~ 0
 ~CTS
 Text GLabel 1750 6400 0    50   Input ~ 0
@@
 Wire Bus Line
 	700  6050 700  7600
+Text Notes 1600 6650 0    50   ~ 0
+08/2023\nCTS RTS swapped to better match my FTDI
 $EndSCHEMATC
