File: KiCad/Rev004/AT_65C02_Computer_Rev004.kicad_pcb (KiCad board)
At the start: 2 copper layers, 241.3 x 149.9 mm, 164 parts, among them J1 CLK Jumper, J11 LCD Connector, J12 System Bus Output port, J14 ESP Interface, J15 Level_Shifter_HV, J16 Level_Shifter_LV, J18 CPU Signals, J2 Optional UART Port, J20 Modem Interface, J21 Expansion port #2, J22 Expansion port #3, J27 LED SWITCH, J29 Decoder Signals, J3 Conn_01x06_Female, J30 Standard Decoder Jumpers, J31 Memory Decoder Expansion, J32 Decoder Expansion, J33 VIA2PA, J4 AudioJack4, J5 Barrel_Jack-Connector, J6 Mini-DIN-6, J7 Expansion port, J8 AVR-ISP-10, J9 VIA2PB, Q1 BC547, SW1 SW_SPDT, SW2 Step, SW3 Mode, SW4 SW_SPDT, U1 74HC21, U10 ATtiny4313-PU, U11 65C22S, U12 65C22S, U13 LM3940, U14 74LS04, U15 74LS08, U16 74LS32, U17 NE555, U18 NE555, U19 NE555, U2 74HC00, U20 74HCT540, U21 74HCT573, U22 74HCT573, U23 74HCT573, U24 10_LED_Array (yellow), U25 10_LED_Array (green), U26 10_LED_Array (red), U27 10_LED_Array (red), U28 LM393, U3 74HC02, U4 NE555, U5 65C51N, U6 Regulator_Linear_L7805, U7 65C02S, U8 28C256, U9 62256, X1 1MHz, X2 1.8432MHz

Commit message: Silkscreen Updates
Routing:
- net a14: track 364.4 -> 363.9 mm

Commit message: minor PCB revisions
Parts:
- added J34: Conn_01x04_Female, Connector_PinSocket_2.54mm:PinSocket_1x04_P2.54mm_Vertical, F.Cu at (226.6, 199.0)
- added J35: Conn_01x03_Male, Connector_PinHeader_2.54mm:PinHeader_1x03_P2.54mm_Vertical, F.Cu at (256.7, 201.8)
- added J36: Conn_01x02_Female, Connector_PinSocket_2.54mm:PinSocket_1x02_P2.54mm_Vertical, F.Cu at (152.7, 147.6)
- J18: footprint Connector_PinSocket_2.54mm:PinSocket_2x07_P2.54mm_Vertical -> Connector_PinSocket_2.54mm:PinSocket_2x08_P2.54mm_Vertical
- moved J2 5.59 mm to (264.5, 196.8)
- moved C7 4.00 mm to (231.8, 199.0)
Connections:
- J14 pad 1: +3.3V -> Net-(J14-Pad1)
- J14 pad 5: +3.3V -> Net-(J14-Pad1)
- J18 pad 13: ~SO -> Net-(J18-Pad13)
- J18 pad 14: BE -> Net-(J18-Pad14)
- J2 pad 1: ~RTS -> ~CTS
- J2 pad 5: ~CTS -> ~RTS
Routing:
- net ~ROM_CS: track 262.3 -> 297.4 mm, vias 7 -> 8
- net Net-(J16-Pad5): track 0.00 -> 27.5 mm
- net Net-(J15-Pad4): track 0.00 -> 15.2 mm
- net Net-(J16-Pad4): track 0.00 -> 15.1 mm
- net Net-(J14-Pad1): track 0.00 -> 12.0 mm
- net Net-(J15-Pad5): track 0.00 -> 11.6 mm
- net GND: track 490.5 -> 483.7 mm
- net TxD: track 93.2 -> 99.6 mm
- net ~RTS: track 35.0 -> 39.4 mm
- net ~ROM_OE: track 98.1 -> 102.4 mm
- net RxD: track 101.0 -> 105.0 mm
- net +3.3V: track 546.9 -> 543.2 mm
- net ~SO: track 43.3 -> 40.0 mm
- net +5V: track 551.5 -> 548.5 mm, vias 14 -> 15
- net BE: track 36.1 -> 33.6 mm
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Other:
- board text added: "H1"
- board text added: "H2"
- board text added: "HI | LO BE"
- board text added: "HI | LO ~SO~"
- board text added: "L1"
- board text added: "L2"
- board text added: "OFF | ON ESP"
- board text added: "~CS"
- board text added: "~OE"
- board text removed: "A3"
- board text removed: "B3"
- board text removed: "B4"
- board text removed: "BE HI | LO"
- board text removed: "~SO~ HI | LO"
